File: kicad/Analogue/Analogue.kicad_pcb (KiCad board)
At the start: 2 copper layers, 4 parts, among them U1 STSPIN220, U2 STSPIN220, U3 STSPIN220, U4 SAM-M8Q

Commit message: Adding libraries
Parts:
- removed the U4 at (86.8, 96.0)
- added U1: BMD-350-A-R, Library:XCVR_BMD-350-A-R, F.Cu at (99.5, 85.0)
- added U5: SAM-M8Q, Library:ublox_SAM-M8Q, F.Cu at (100.0, 110.0)
- moved U4 14.3 mm to (112.0, 92.5)
- moved U2 12.6 mm to (86.0, 94.0)
- moved U3 9.17 mm to (94.5, 92.5)
- renumbered U1 to U4
Other:
- board outline added: 40 x 40 mm
