File: kicad/Analogue/Analogue.kicad_sch (KiCad schematic)
At the start: 4 parts, among them U1 STSPIN220, U2 STSPIN220, U3 STSPIN220, U4 SAM-M8Q

Commit message: Adding libraries
Parts:
- removed U4: SAM-M8Q, RF_GPS:ublox_SAM-M8Q, symbol RF_GPS:SAM-M8Q
- added U1: BMD-350-A-R, XCVR_BMD-350-A-R, symbol Analogue:BMD-350-A-R
- added U5: SAM-M8Q, Library:ublox_SAM-M8Q, symbol RF_GPS:SAM-M8Q
- renumbered U1 to U4
Connections:
- new net: U1.1 (GND), U1.15 (GND), U1.2 (GND), U1.26 (GND), U1.3 (GND), U1.37 (GND), U1.38 (GND), U1.39 (GND), U1.40 (GND), U1.43 (GND), U1.46 (GND), U1.47 (GND)
- new net: U5.1 (GND), U5.10 (GND), U5.11 (GND), U5.15 (GND), U5.16 (GND), U5.20 (GND), U5.4 (GND), U5.5 (GND), U5.6 (GND)
Other:
- moved on the sheet: U4
Changed lines of the file:
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@@
 (kicad_sch (version 20211123) (generator eeschema)
   (paper "A4")
-  (symbol (lib_id "RF_GPS:SAM-M8Q") (at 55.88 33.02 0) (unit 1)
-    (in_bom yes) (on_board yes) (fields_autoplaced)
-    (property "Reference" "U4" (id 0) (at 57.8994 45.72 0)
-      (effects (font (size 1.27 1.27)) (justify left))
-    )
-    (property "Value" "SAM-M8Q" (id 1) (at 57.8994 48.26 0)
-      (effects (font (size 1.27 1.27)) (justify left))
-    )
-    (property "Footprint" "RF_GPS:ublox_SAM-M8Q" (id 2) (at 68.58 44.45 0)
-      (effects (font (size 1.27 1.27)) hide)
-    )
-    (property "Datasheet" "https://www.u-blox.com/sites/default/files/SAM-M8Q_DataSheet_%28UBX-16012619%29.pdf" (id 3) (at 55.88 33.02 0)
-      (effects (font (size 1.27 1.27)) hide)
+  (symbol (lib_id "Analogue:BMD-350-A-R") (at 215.9 63.5 0) (unit 1)
+    (in_bom yes) (on_board yes) (fields_autoplaced)
+    (property "Reference" "U1" (id 0) (at 215.9 25.4 0))
+    (property "Value" "BMD-350-A-R" (id 1) (at 215.9 27.94 0))
+    (property "Footprint" "XCVR_BMD-350-A-R" (id 2) (at 215.9 63.5 0)
+      (effects (font (size 1.27 1.27)) (justify left bottom) hide)
+    )
+    (property "Datasheet" "" (id 3) (at 215.9 63.5 0)
+      (effects (font (size 1.27 1.27)) (justify left bottom) hide)
+    )
+    (property "STANDARD" "Manufacturer Recommendations" (id 4) (at 215.9 63.5 0)
+      (effects (font (size 1.27 1.27)) (justify left bottom) hide)
+    )
+    (property "PARTREV" "2.0" (id 5) (at 215.9 63.5 0)
+      (effects (font (size 1.27 1.27)) (justify left bottom) hide)
+    )
+    (property "MANUFACTURER" "RIGADO" (id 6) (at 215.9 63.5 0)
+      (effects (font (size 1.27 1.27)) (justify left bottom) hide)
     )
     (pin "1")
@@
     (pin "2")
     (pin "20")
-    (pin "3")
-    (pin "4")
+    (pin "21")
+    (pin "22")
+    (pin "23")
+    (pin "24")
+    (pin "25")
+    (pin "26")
+    (pin "27")
+    (pin "28")
+    (pin "29")
+    (pin "3")
+    (pin "30")
+    (pin "31")
+    (pin "32")
+    (pin "33")
+    (pin "34")
+    (pin "35")
+    (pin "36")
+    (pin "37")
+    (pin "38")
+    (pin "39")
+    (pin "4")
+    (pin "40")
+    (pin "41")
+    (pin "42")
+    (pin "43")
+    (pin "44")
+    (pin "45")
+    (pin "46")
+    (pin "47")
     (pin "5")
     (pin "6")
@@
     (pin "9")
   )
-  (symbol (lib_id "Driver_Motor:STSPIN220") (at 36.83 105.41 0) (unit 1)
-    (in_bom yes) (on_board yes) (fields_autoplaced)
-    (property "Reference" "U1" (id 0) (at 38.8494 85.09 0)
-      (effects (font (size 1.27 1.27)) (justify left))
-    )
-    (property "Value" "STSPIN220" (id 1) (at 38.8494 87.63 0)
-      (effects (font (size 1.27 1.27)) (justify left))
-    )
-    (property "Footprint" "Package_DFN_QFN:VQFN-16-1EP_3x3mm_P0.5mm_EP1.8x1.8mm" (id 2) (at 41.91 86.36 0)
+  (symbol (lib_id "RF_GPS:SAM-M8Q") (at 63.5 63.5 0) (unit 1)
+    (in_bom yes) (on_board yes) (fields_autoplaced)
+    (property "Reference" "U5" (id 0) (at 65.5194 76.2 0)
+      (effects (font (size 1.27 1.27)) (justify left))
+    )
+    (property "Value" "SAM-M8Q" (id 1) (at 65.5194 78.74 0)
+      (effects (font (size 1.27 1.27)) (justify left))
+    )
+    (property "Footprint" "Library:ublox_SAM-M8Q" (id 2) (at 76.2 74.93 0)
+      (effects (font (size 1.27 1.27)) hide)
+    )
+    (property "Datasheet" "https://www.u-blox.com/sites/default/files/SAM-M8Q_DataSheet_%28UBX-16012619%29.pdf" (id 3) (at 63.5 63.5 0)
+      (effects (font (size 1.27 1.27)) hide)
+    )
+    (pin "1")
+    (pin "10")
+    (pin "11")
+    (pin "12")
+    (pin "13")
+    (pin "14")
+    (pin "15")
+    (pin "16")
+    (pin "17")
+    (pin "18")
+    (pin "19")
+    (pin "2")
+    (pin "20")
+    (pin "3")
+    (pin "4")
+    (pin "5")
+    (pin "6")
+    (pin "7")
+    (pin "8")
+    (pin "9")
+  )
+  (symbol (lib_id "Driver_Motor:STSPIN220") (at 74.93 147.32 0) (unit 1)
+    (in_bom yes) (on_board yes) (fields_autoplaced)
+    (property "Reference" "U4" (id 0) (at 76.9494 127 0)
+      (effects (font (size 1.27 1.27)) (justify left))
+    )
+    (property "Value" "STSPIN220" (id 1) (at 76.9494 129.54 0)
+      (effects (font (size 1.27 1.27)) (justify left))
+    )
+    (property "Footprint" "Package_DFN_QFN:VQFN-16-1EP_3x3mm_P0.5mm_EP1.8x1.8mm" (id 2) (at 80.01 128.27 0)
       (effects (font (size 1.27 1.27)) (justify left) hide)
     )
-    (property "Datasheet" "www.st.com/resource/en/datasheet/stspin220.pdf" (id 3) (at 40.64 99.06 0)
+    (property "Datasheet" "www.st.com/resource/en/datasheet/stspin220.pdf" (id 3) (at 78.74 140.97 0)
       (effects (font (size 1.27 1.27)) hide)
     )
@@
   )
   (symbol_instances
-    (path "/d2b2d451-8d34-4eda-8b46-20ceba6fc80f"
-      (reference "U1") (unit 1) (value "STSPIN220") (footprint "Package_DFN_QFN:VQFN-16-1EP_3x3mm_P0.5mm_EP1.8x1.8mm")
+    (path "/57c1bafc-a5fb-4034-9d60-a13a4b79ea51"
+      (reference "U1") (unit 1) (value "BMD-350-A-R") (footprint "XCVR_BMD-350-A-R")
     )
     (path "/76dd8502-ef22-4ccd-b6b2-35d3f171bae0"
@@
       (reference "U3") (unit 1) (value "STSPIN220") (footprint "Package_DFN_QFN:VQFN-16-1EP_3x3mm_P0.5mm_EP1.8x1.8mm")
     )
-    (path "/3487b883-d132-4810-af37-6ee3794b3652"
-      (reference "U4") (unit 1) (value "SAM-M8Q") (footprint "RF_GPS:ublox_SAM-M8Q")
-    )
-  )
+    (path "/d2b2d451-8d34-4eda-8b46-20ceba6fc80f"
+      (reference "U4") (unit 1) (value "STSPIN220") (footprint "Package_DFN_QFN:VQFN-16-1EP_3x3mm_P0.5mm_EP1.8x1.8mm")
+    )
+    (path "/9af95414-3aef-4e69-b371-7ccc1a849afe"
+      (reference "U5") (unit 1) (value "SAM-M8Q") (footprint "Library:ublox_SAM-M8Q")
+    )
+  )
